Commit message: Added the controller by joystick

File: components/pybullet_bump/URDFs/shadow/shadow.urdf (robot description, URDF)
Before this commit: robot shadow_ahiora_si_definivo_okok, 16 links, 15 joints
Joints:
- joint frame_back_left2motor_back_left: axis 0 1 0 -> 0 -1 0
- joint frame_back_right2motor_back_right: axis 0 -1 0 -> 0 1 0
