Commit message: Trying the loop of bumps

File: components/pybullet_bump/URDFs/bump/cylinder_bump_10m.urdf (robot description, URDF)
Before this commit: robot bump_100x5, 1 links, 0 joints
Links:
- link base_link: geometry collision mesh filename=cylinder_bump_10m.stl scale=1 1 0.5; visual mesh filename=cylinder_bump_10m.stl scale=1 1 0.5
